File: Source/KiCad - PCB/Plant Buddy/Plant Buddy.kicad_pcb (KiCad board)
At the start: 2 copper layers, 80 x 80 mm, 36 parts, among them J1 Screw_Terminal_01x02, J2 Conn_01x03, J3 Conn_02x04_Counter_Clockwise, Q1 AO3401, SW2 (EN), U1 AMS1117-3.3, U2 TLC555xD

Commit message: Edited PCB and schematics.
Connections:
- J3 pad 4: unconnected-(J3-Pin_4-Pad4) -> GPIO25
- Q1 pad 3: V3.3 -> VBUS
- U4 pad 8: unconnected-(U4-IO25-Pad8) -> GPIO25
Routing:
- net GPIO25: track 0.00 -> 77.3 mm, vias 0 -> 2
- net V3.3: track 147.4 -> 104.3 mm, vias 6 -> 4
- net VBUS: track 176.3 -> 196.0 mm, vias 5 -> 7

Commit message: Finished the firmware and modified the schematics and the PCB
Parts:
- added R10: 220, Resistor_SMD:R_0805_2012Metric_Pad1.20x1.40mm_HandSolder, F.Cu at (156.9, 93.8)
- added U3: PC817, Package_DIP:DIP-4_W7.62mm, F.Cu at (153.1, 97.8)
- moved Q1 1.47 mm to (165.6, 99.4)
Connections:
- Q1 pad 1: GPIO5 -> Net-(Q1-G)
- Q1 pad 2: Net-(J1-Pin_1) -> VBUS
- Q1 pad 3: VBUS -> Net-(J1-Pin_1)
Routing:
- net VBUS: track 196.0 -> 206.0 mm
- net GPIO25: track 77.3 -> 70.3 mm
- net Net-(R10-Pad2): track 0.00 -> 6.40 mm, vias 0 -> 1
- net Net-(Q1-G): track 0.00 -> 4.62 mm
- net Net-(J1-Pin_1): track 15.0 -> 11.3 mm
- net GPIO5: track 65.1 -> 68.5 mm

Commit message: Designed 3D case
Connections:
- J2 pad 2: Net-(J2-Pin_2) -> VBUS
- J2 pad 3: VBUS -> Net-(J2-Pin_3)
- R7 pad 1: Net-(J2-Pin_2) -> Net-(J2-Pin_3)
Routing:
- net VBUS: track 206.0 -> 229.1 mm
- net Net-(J2-Pin_2): track 13.5 -> 0.00 mm, vias 1 -> 0
- net Net-(J2-Pin_3): track 0.00 -> 11.2 mm, vias 0 -> 1
- net GND: track 210.8 -> 216.9 mm
- net VBAT: track 89.1 -> 85.6 mm
- net Net-(U4-EN): vias 2 -> 1
